File: kicad/keyboard.kicad_pcb (KiCad board)
At the start: 2 copper layers, 169 parts, among them SW1 Push, SW10 Push, SW11 Push, SW12 Push, SW13 Push, SW14 Push, SW15 Push, SW16 Push, SW17 Push, SW18 Push, SW19 Push, SW2 Push, SW20 Push, SW21 Push, SW22 Push, SW23 Push, SW24 Push, SW25 Push, SW26 Push, SW27 Push, SW28 Push, SW29 Push, SW3 Push, SW30 Push, SW31 Push, SW32 Push, SW33 Push, SW34 Push, SW35 Push, SW36 Push, SW37 Push, SW38 Push, SW39 Push, SW4 Push, SW40 Push, SW41 Push, SW42 Push, SW43 Push, SW44 Push, SW45 Push, SW46 Push, SW47 Push, SW48 Push, SW49 Push, SW5 Push, SW50 Push, SW51 Push, SW52 Push, SW53 Push, SW54 Push, SW55 Push, SW56 Push, SW57 Push, SW58 Push, SW59 Push, SW6 Push, SW60 Push, SW61 Push, SW62 Push, SW63 Push, SW64 Push, SW65 Push, SW66 Push, SW67 Push, SW68 Push, SW69 Push, SW7 Push, SW70 Push, SW71 Push, SW72 Push, SW73 Push, SW74 Push, SW75 Push, SW76 Push, SW77 Push, SW78 Push, SW79 Push, SW8 Push, SW80 Push, SW81 Push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

Commit message: gi2
Routing:
- net Net-(D1-A): track 0.00 -> 5.15 mm
Changed lines of the file:
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@@
 		(at 37.375 33.4)
 		(property "Reference" "SW1"
-			(at 0 -3.5 360)
+			(at 0 -3.5 0)
 			(layer "Dwgs.User")
 			(effects
@@
 		)
 		(property "Value" "Push"
-			(at 0 -7.9375 360)
+			(at 0 -7.9375 0)
 			(layer "Dwgs.User")
 			(effects
@@
 		)
 	)
+	(segment
+		(start 27.85 38.1625)
+		(end 32.9125 38.1625)
+		(width 0.2)
+		(layer "B.Cu")
+		(net 1)
+	)
+	(segment
+		(start 32.9125 38.1625)
+		(end 32.975 38.1)
+		(width 0.2)
+		(layer "B.Cu")
+		(net 1)
+	)
 )

Commit message: traces
Parts:
- moved U1 3.70 mm to (9.44, 49.9)
Routing:
- net ROW5: track 0.00 -> 339.6 mm, vias 0 -> 14
- net ROW3: track 0.00 -> 339.6 mm, vias 0 -> 14
- net ROW2: track 0.00 -> 339.6 mm, vias 0 -> 14
- net ROW1: track 0.00 -> 339.6 mm, vias 0 -> 14
- net ROW0: track 0.00 -> 339.6 mm, vias 0 -> 14
- net ROW4: track 0.00 -> 339.6 mm, vias 0 -> 14
- net COL1: track 0.00 -> 138.6 mm
- net COL3: track 0.00 -> 133.8 mm
- net COL2: track 0.00 -> 133.8 mm
- net COL4: track 0.00 -> 133.1 mm
- net COL0: track 0.00 -> 129.7 mm
- net COL7: track 0.00 -> 129.0 mm
- net COL13: track 0.00 -> 129.0 mm
- net COL12: track 0.00 -> 129.0 mm
- net COL8: track 0.00 -> 129.0 mm
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
Commit message: pi traces
Parts:
- moved SW10 78.1 mm to (118.3, 138.2)
- moved SW28 78.1 mm to (175.5, 138.2)
- moved SW55 78.1 mm to (270.7, 81.0)
- moved SW58 78.1 mm to (270.7, 138.2)
- moved SW61 78.1 mm to (289.8, 81.0)
- moved SW64 78.1 mm to (289.8, 138.2)
- moved SW79 78.1 mm to (346.9, 81.0)
- moved SW82 78.1 mm to (346.9, 138.2)
- moved D25 78.1 mm to (166.0, 84.1)
- moved D26 78.1 mm to (166.0, 103.2)
- moved D27 78.1 mm to (166.0, 122.2)
- moved D28 78.1 mm to (166.0, 141.3)
- moved D29 78.1 mm to (166.0, 160.3)
- moved D30 78.1 mm to (166.0, 179.4)
- moved D43 78.1 mm to (223.1, 84.1)
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Connections:
- U1 pad 19: ROW0 -> unconnected-(U1-GPIO14-Pad19)
- U1 pad 20: ROW1 -> unconnected-(U1-GPIO15-Pad20)
- U1 pad 21: ROW2 -> ROW5
- U1 pad 22: ROW3 -> ROW4
- U1 pad 24: ROW4 -> ROW3
- U1 pad 25: ROW5 -> ROW2
- U1 pad 26: unconnected-(U1-GPIO20-Pad26) -> ROW1
- U1 pad 27: unconnected-(U1-GPIO21-Pad27) -> ROW0
- U1 pad 3: COL2 -> unconnected-(U1-GND-Pad3)
Routing:
- net COL13: track 129.0 -> 409.5 mm
- net COL12: track 129.0 -> 392.5 mm
- net COL11: track 129.0 -> 375.6 mm
- net COL10: track 129.0 -> 358.3 mm
- net COL9: track 129.0 -> 343.7 mm
- net COL8: track 129.0 -> 326.5 mm
- net COL7: track 129.0 -> 309.4 mm
- net COL6: track 129.0 -> 292.3 mm
- net COL5: track 129.0 -> 277.6 mm
- net COL4: track 133.1 -> 264.5 mm
- net ROW5: track 339.6 -> 464.4 mm
- net COL3: track 133.8 -> 248.0 mm
- net ROW0: track 339.6 -> 448.9 mm
- net ROW4: track 339.6 -> 442.5 mm
- net COL2: track 133.8 -> 230.8 mm
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
Commit message: outline
Routing:
- net (no net): track 9.53 -> 0.00 mm
Other:
- board outline added: 304.5 x 124 mm
