File: kicad/keyboard.kicad_pcb (KiCad board)
At the start: 2 copper layers, 304.5 x 124 mm, 169 parts, among them SW1 Push, SW10 Push, SW11 Push, SW12 Push, SW13 Push, SW14 Push, SW15 Push, SW16 Push, SW17 Push, SW18 Push, SW19 Push, SW2 Push, SW20 Push, SW21 Push, SW22 Push, SW23 Push, SW24 Push, SW25 Push, SW26 Push, SW27 Push, SW28 Push, SW29 Push, SW3 Push, SW30 Push, SW31 Push, SW32 Push, SW33 Push, SW34 Push, SW35 Push, SW36 Push, SW37 Push, SW38 Push, SW39 Push, SW4 Push, SW40 Push, SW41 Push, SW42 Push, SW43 Push, SW44 Push, SW45 Push, SW46 Push, SW47 Push, SW48 Push, SW49 Push, SW5 Push, SW50 Push, SW51 Push, SW52 Push, SW53 Push, SW54 Push, SW55 Push, SW56 Push, SW57 Push, SW58 Push, SW59 Push, SW6 Push, SW60 Push, SW61 Push, SW62 Push, SW63 Push, SW64 Push, SW65 Push, SW66 Push, SW67 Push, SW68 Push, SW69 Push, SW7 Push, SW70 Push, SW71 Push, SW72 Push, SW73 Push, SW74 Push, SW75 Push, SW76 Push, SW77 Push, SW78 Push, SW79 Push, SW8 Push, SW80 Push, SW81 Push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

Commit message: filled zone
Routing:
- added copper zone on B.Cu, net (none)
- added copper zone on F.Cu, net (none)
Changed lines of the file:
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@@
 		(net 104)
+	)
+	(zone
+		(net 0)
+		(net_name "")
+		(layers "F&B.Cu")
+		(hatch edge 0.5)
+		(connect_pads
+			(clearance 0.5)
+		)
+		(min_thickness 0.25)
+		(filled_areas_thickness no)
+		(fill yes
+			(thermal_gap 0.5)
+			(thermal_bridge_width 0.5)
+			(island_removal_mode 1)
+			(island_area_min 10)
+		)
+		(polygon
+			(pts
+				(xy 44.7625 51.5) (xy 364.7625 51.5) (xy 364.7625 201.5) (xy 44.7625 201.5)
+			)
+		)
 	)
 	(group ""

Commit message: init
Parts:
- removed D13, D19, D25, D31, D37, D43, D49, D55, D61, D67, D7, D73, D74, D75, D76, D77, D78, D80, D81, D82, D83, D84: 1N47xxA, ScottoKeebs_Components:Diode_SOD-123
- removed SW13, SW19, SW25, SW31, SW37, SW43, SW49, SW55, SW61, SW67, SW7, SW73, SW74, SW75, SW76, SW77, SW78, SW80, SW81, SW82, SW83, SW84: Push, Gateron_KS33_Solderable:Gateron-KS33-Solderable-1U
- SW1, SW10, SW11, SW12, SW14, SW15, SW16, SW17, SW18, SW2, SW20, SW21, SW22, SW23, SW24, SW26, SW27, SW28, SW29, SW3, SW30, SW32, SW33, SW34, SW35, SW36, SW38, SW39, SW4, SW40, SW41, SW42, SW44, SW45, SW46, SW47, SW48, SW5, SW50, SW51, SW52, SW53, SW54, SW56, SW57, SW58, SW59, SW6, SW60, SW62, SW63, SW64, SW65, SW66, SW68, SW69, SW70, SW71, SW72, SW79, SW8, SW9: footprint Gateron_KS33_Solderable:Gateron-KS33-Solderable-1U -> ScottoKeebs_Hotswap:Hotswap_Choc_V1_1.00u
- U1: value Raspberry_Pi_Pico -> Arduino_Pro_Micro; footprint ScottoKeebs_MCU:Raspberry_Pi_Pico -> ScottoKeebs_MCU:Arduino_Pro_Micro
- moved U1 154.8 mm to (225.3, 80.1), turned to 90 degrees
- moved SW79 38.1 mm to (308.8, 81.0)
- moved D79 32.2 mm to (305.3, 85.8), turned to 90 degrees
- moved D20 6.32 mm to (152.9, 105.3), turned to 90 degrees
- moved D14 6.18 mm to (133.8, 104.8), turned to 90 degrees
- moved D15 6.18 mm to (133.8, 123.9), turned to 90 degrees
- moved D16 6.18 mm to (133.8, 142.9), turned to 90 degrees
- moved D17 6.18 mm to (133.8, 162.0), turned to 90 degrees
- moved D18 6.18 mm to (133.8, 181.0), turned to 90 degrees
- moved D10 6.18 mm to (114.8, 142.9), turned to 90 degrees
- moved D11 6.18 mm to (114.8, 162.0), turned to 90 degrees
- moved D12 6.18 mm to (114.8, 181.0), turned to 90 degrees
- moved D2 6.18 mm to (95.7, 104.8), turned to 90 degrees
- moved D21 6.18 mm to (152.9, 123.9), turned to 90 degrees
- moved D22 6.18 mm to (152.9, 142.9), turned to 90 degrees
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Connections:
- D79 pad 2: Net-(D79-A) -> COL11
- SW79 pad 1: Net-(D79-A) -> COL11
- SW79 pad 2: COL13 -> COL11
- U1 pad 1: COL0 -> COL5
- U1 pad 11: COL8 -> COL9
- U1 pad 12: COL9 -> COL8
- U1 pad 13: unconnected-(U1-GND-Pad13) -> COL11
- U1 pad 15: COL11 -> ROW2
- U1 pad 16: COL12 -> ROW1
- U1 pad 17: COL13 -> ROW0
- U1 pad 18: unconnected-(U1-GND-Pad18) -> ROW3
- U1 pad 19: unconnected-(U1-GPIO14-Pad19) -> ROW4
- U1 pad 2: COL1 -> COL4
- U1 pad 20: unconnected-(U1-GPIO15-Pad20) -> ROW5
- U1 pad 21: ROW5 -> unconnected-(U1-VCC-Pad21)
- U1 pad 22: ROW4 -> unconnected-(U1-RST-Pad22)
- U1 pad 24: ROW3 -> unconnected-(U1-RAW-Pad24)
- U1 pad 4: COL2 -> unconnected-(U1-GND-Pad4)
- U1 pad 6: COL4 -> COL2
- U1 pad 7: COL5 -> COL1
- U1 pad 8: unconnected-(U1-GND-Pad8) -> COL0
Routing:
- net COL13: track 409.5 -> 0.00 mm
- net COL12: track 392.5 -> 0.00 mm
- net COL8: track 326.5 -> 103.0 mm
- net COL7: track 309.4 -> 90.1 mm
- net COL9: track 343.7 -> 126.8 mm
- net ROW0: track 448.9 -> 241.2 mm, vias 14 -> 2
- net COL10: track 358.3 -> 155.5 mm
- net COL6: track 292.3 -> 92.7 mm
- net COL5: track 277.6 -> 90.2 mm
- net COL11: track 375.6 -> 196.9 mm
- net COL4: track 264.5 -> 114.5 mm
- net COL3: track 248.0 -> 141.1 mm
- net COL2: track 230.8 -> 163.1 mm
- net ROW1: track 433.8 -> 370.5 mm, vias 14 -> 12
- net COL1: track 220.9 -> 186.2 mm
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- removed copper zone on B.Cu, net (none)
- removed copper zone on F.Cu, net (none)
Other:
- board size 304.5 x 124 mm -> 231 x 116.7 mm

Commit message: S67 fix
Parts:
- renumbered D79 to D67, SW79 to SW67
Connections:
- D67 pad 2: COL11 -> Net-(D67-A)
- SW67 pad 1: COL11 -> Net-(D67-A)
Routing:
- net COL11: track 196.9 -> 187.7 mm
- net Net-(D67-A): track 0.00 -> 9.14 mm
Changed lines of the file:
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@@
 	(net 82 "unconnected-(U1-RST-Pad22)")
 	(net 83 "unconnected-(U1-GND-Pad4)")
-	(net 84 "unconnected-(U1-GND-Pad23)")
-	(net 85 "unconnected-(U1-GND-Pad3)")
+	(net 84 "Net-(D67-A)")
+	(net 85 "unconnected-(U1-GND-Pad23)")
+	(net 86 "unconnected-(U1-GND-Pad3)")
 	(footprint "ScottoKeebs_Hotswap:Hotswap_Choc_V1_1.00u"
 		(layer "F.Cu")
@@
 		(descr "Choc keyswitch V1 CPG1350 V1 Hotswap Keycap 1.00u")
 		(tags "Choc Keyswitch Switch CPG1350 V1 Hotswap Cutout Keycap 1.00u")
-		(property "Reference" "SW79"
+		(property "Reference" "SW67"
 			(at 0 -9 0)
 			(layer "F.SilkS")
@@
 			(layers "B.Cu" "B.Paste" "B.Mask")
 			(roundrect_rratio 0.1)
-			(net 81 "COL11")
+			(net 84 "Net-(D67-A)")
 			(pinfunction "1")
 			(pintype "passive")
@@
 			(layers "*.Cu" "*.SilkS" "*.Mask")
 			(remove_unused_layers no)
-			(net 85 "unconnected-(U1-GND-Pad3)")
+			(net 86 "unconnected-(U1-GND-Pad3)")
 			(pinfunction "GND")
 			(pintype "input")
@@
 			(layers "*.Cu" "*.SilkS" "*.Mask")
 			(remove_unused_layers no)
-			(net 84 "unconnected-(U1-GND-Pad23)")
+			(net 85 "unconnected-(U1-GND-Pad23)")
 			(pinfunction "GND")
 			(pintype "input")
@@
 	(footprint "ScottoKeebs_Components:Diode_SOD-123"
 		(layer "B.Cu")
-		(at 305.265625 85.7875 90)
+		(at 305.265444 85.787488 90)
 		(descr "SOD-123")
 		(tags "SOD-123")
-		(property "Reference" "D79"
+		(property "Reference" "D67"
 			(at 0 2 90)
 			(layer "B.SilkS")
@@
 			(layers "B.Cu" "B.Paste" "B.Mask")
 			(roundrect_rratio 0.25)
-			(net 81 "COL11")
+			(net 84 "Net-(D67-A)")
 			(pinfunction "A")
 			(pintype "passive")
@@
 	)
 	(segment
-		(start 305.265625 87.4375)
+		(start 305.265444 87.437488)
+		(end 305.265444 90.549819)
+		(width 0.2)
+		(layer "B.Cu")
+		(net 2)
+	)
+	(segment
+		(start 305.265444 90.549819)
 		(end 305.265625 90.55)
 		(width 0.2)
@@
 	)
 	(segment
-		(start 246.72646 89.657016)
-		(end 239.285059 82.215615)
+		(start 296.63342 89.657016)
+		(end 246.72646 89.657016)
 		(width 0.2)
 		(layer "B.Cu")
@@
 	(segment
 		(start 317.3375 91.740608)
-		(end 317.3375 77.225)
+		(end 298.717012 91.740608)
 		(width 0.2)
 		(layer "B.Cu")
@@
 	)
 	(segment
-		(start 317.3375 172.475)
-		(end 317.3375 96.275)
-		(width 0.2)
-		(layer "B.Cu")
-		(net 81)
-	)
-	(segment
-		(start 296.63342 89.657016)
-		(end 246.72646 89.657016)
+		(start 239.285059 82.215615)
+		(end 239.285059 71.797656)
 		(width 0.2)
 		(layer "B.Cu")
@@
 	)
 	(segment
-		(start 305.3375 84.065625)
-		(end 305.265625 84.1375)
+		(start 298.717012 91.740608)
+		(end 296.63342 89.657016)
 		(width 0.2)
 		(layer "B.Cu")
@@
 	)
 	(segment
-		(start 305.3375 75.025)
-		(end 305.3375 84.065625)
+		(start 239.285059 71.797656)
+		(end 239.225515 71.738112)
 		(width 0.2)
 		(layer "B.Cu")
@@
 	)
 	(segment
-		(start 317.3375 96.275)
-		(end 317.3375 91.740608)
+		(start 317.3375 91.740608)
+		(end 317.3375 77.225)
 		(width 0.2)
 		(layer "B.Cu")
@@
 	)
 	(segment
-		(start 298.6875 91.711096)
-		(end 296.63342 89.657016)
+		(start 317.3375 172.475)
+		(end 317.3375 96.275)
 		(width 0.2)
 		(layer "B.Cu")
@@
 	)
 	(segment
-		(start 317.3375 91.740608)
-		(end 298.6875 91.740608)
+		(start 246.72646 89.657016)
+		(end 239.285059 82.215615)
 		(width 0.2)
 		(layer "B.Cu")
@@
 	)
 	(segment
-		(start 298.6875 91.740608)
-		(end 298.6875 91.711096)
+		(start 317.3375 96.275)
+		(end 317.3375 91.740608)
 		(width 0.2)
 		(layer "B.Cu")
@@
 	)
 	(segment
-		(start 239.285059 71.797656)
-		(end 239.225515 71.738112)
+		(start 305.3375 75.025)
+		(end 305.3375 84.065432)
 		(width 0.2)
 		(layer "B.Cu")
-		(net 81)
+		(net 84)
 	)
 	(segment
-		(start 239.285059 82.215615)
-		(end 239.285059 71.797656)
+		(start 305.3375 84.065432)
+		(end 305.265444 84.137488)
 		(width 0.2)
 		(layer "B.Cu")
-		(net 81)
+		(net 84)
 	)
 	(group ""

Commit message: path tweaks
Routing:
- net COL0: track 225.5 -> 220.9 mm
- net COL9: track 126.8 -> 128.6 mm
- net COL10: track 155.5 -> 156.6 mm
