File: kicad/keyboard.kicad_pcb (KiCad board)
At the start: 2 copper layers, 231 x 116.7 mm, 125 parts, among them SW1 Push, SW10 Push, SW11 Push, SW12 Push, SW14 Push, SW15 Push, SW16 Push, SW17 Push, SW18 Push, SW2 Push, SW20 Push, SW21 Push, SW22 Push, SW23 Push, SW24 Push, SW26 Push, SW27 Push, SW28 Push, SW29 Push, SW3 Push, SW30 Push, SW32 Push, SW33 Push, SW34 Push, SW35 Push, SW36 Push, SW38 Push, SW39 Push, SW4 Push, SW40 Push, SW41 Push, SW42 Push, SW44 Push, SW45 Push, SW46 Push, SW47 Push, SW48 Push, SW5 Push, SW50 Push, SW51 Push, SW52 Push, SW53 Push, SW54 Push, SW56 Push, SW57 Push, SW58 Push, SW59 Push, SW6 Push, SW60 Push, SW62 Push, SW63 Push, SW64 Push, SW65 Push, SW66 Push, SW67 Push, SW68 Push, SW69 Push, SW70 Push, SW71 Push, SW72 Push, SW8 Push, SW9 Push, U1 Arduino_Pro_Micro

Commit message: spacebar
Parts:
- removed D36: 1N47xxA, ScottoKeebs_Components:Diode_SOD-123
- removed SW36: Push, ScottoKeebs_Hotswap:Hotswap_Choc_V1_1.00u
- moved D42 9.53 mm to (200.5, 181.0)
- moved SW42 9.53 mm to (204.1, 176.3)
Routing:
- net COL5: track 90.2 -> 71.2 mm
- net COL6: track 92.7 -> 102.3 mm
- net Net-(D36-A): track 9.14 -> 0.00 mm
- net ROW5: track 487.7 -> 484.6 mm, vias 12 -> 11

Commit message: case v1
Other:
- board size 231 x 116.7 mm -> 232.6 x 118.3 mm
Changed lines of the file:
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@@
 	)
 	(gr_line
-		(start 88.571875 183.990625)
-		(end 88.571875 73.309375)
+		(start 87.7625 183.990618)
+		(end 87.7625 73.309368)
+		(stroke
+			(width 0.05)
+			(type default)
+		)
+		(layer "Edge.Cuts")
+	)
+	(gr_circle
+		(center 294.55 81.025)
+		(end 295.6 81.025)
+		(stroke
+			(width 0.05)
+			(type default)
+		)
+		(fill none)
+		(layer "Edge.Cuts")
+	)
+	(gr_circle
+		(center 113.575 81.025)
+		(end 114.625 81.025)
+		(stroke
+			(width 0.05)
+			(type default)
+		)
+		(fill none)
+		(layer "Edge.Cuts")
+	)
+	(gr_circle
+		(center 204.0625 159.60625)
+		(end 205.1125 159.60625)
+		(stroke
+			(width 0.05)
+			(type default)
+		)
+		(fill none)
+		(layer "Edge.Cuts")
+	)
+	(gr_arc
+		(start 320.3625 183.990631)
+		(mid 319.246748 186.684257)
+		(end 316.553118 187.8)
+		(stroke
+			(width 0.05)
+			(type default)
+		)
+		(layer "Edge.Cuts")
+	)
+	(gr_circle
+		(center 299.312324 178.65625)
+		(end 300.362324 178.65625)
+		(stroke
+			(width 0.05)
+			(type default)
+		)
+		(fill none)
+		(layer "Edge.Cuts")
+	)
+	(gr_line
+		(start 91.571875 69.5)
+		(end 316.553125 69.5)
 		(stroke
 			(width 0.05)
@@
 	)
 	(gr_arc
-		(start 319.553125 183.990625)
-		(mid 318.674445 186.111945)
-		(end 316.553125 186.990625)
+		(start 87.7625 73.309368)
+		(mid 88.87825 70.615745)
+		(end 91.571875 69.5)
 		(stroke
 			(width 0.05)
@@
 	)
 	(gr_line
-		(start 91.571875 70.309375)
-		(end 316.553125 70.309375)
+		(start 316.553118 187.8)
+		(end 91.571868 187.8)
 		(stroke
 			(width 0.05)
@@
 	)
 	(gr_arc
-		(start 88.571875 73.309375)
-		(mid 89.450562 71.188062)
-		(end 91.571875 70.309375)
+		(start 316.553132 69.5)
+		(mid 319.246757 70.615752)
+		(end 320.3625 73.309381)
 		(stroke
 			(width 0.05)
@@
 	)
 	(gr_line
-		(start 316.553125 186.990625)
-		(end 91.571875 186.990625)
+		(start 320.3625 73.309381)
+		(end 320.3625 183.990631)
 		(stroke
 			(width 0.05)
@@
 		(layer "Edge.Cuts")
 	)
-	(gr_arc
-		(start 316.553125 70.309375)
-		(mid 318.674445 71.188055)
-		(end 319.553125 73.309375)
+	(gr_circle
+		(center 108.812484 178.65625)
+		(end 109.862484 178.65625)
 		(stroke
 			(width 0.05)
 			(type default)
 		)
-		(layer "Edge.Cuts")
-	)
-	(gr_line
-		(start 319.553125 73.309375)
-		(end 319.553125 183.990625)
-		(stroke
-			(width 0.05)
-			(type default)
-		)
+		(fill none)
 		(layer "Edge.Cuts")
 	)
 	(gr_arc
-		(start 91.571875 186.990625)
-		(mid 89.450555 186.111945)
-		(end 88.571875 183.990625)
+		(start 91.571868 187.8)
+		(mid 88.878242 186.684248)
+		(end 87.7625 183.990618)
 		(stroke
 			(width 0.05)

Commit message: case v2
Routing:
- net COL8: track 103.0 -> 105.3 mm
- net COL2: track 163.1 -> 165.4 mm
Other:
- outline, holes or cut-outs redrawn
Changed lines of the file:
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@@
 	)
 	(gr_circle
-		(center 294.55 81.025)
-		(end 295.6 81.025)
-		(stroke
-			(width 0.05)
-			(type default)
-		)
-		(fill none)
-		(layer "Edge.Cuts")
-	)
-	(gr_circle
-		(center 113.575 81.025)
-		(end 114.625 81.025)
-		(stroke
-			(width 0.05)
-			(type default)
-		)
-		(fill none)
-		(layer "Edge.Cuts")
-	)
-	(gr_circle
-		(center 204.0625 159.60625)
-		(end 205.1125 159.60625)
+		(center 261.212356 107.516376)
+		(end 262.262356 107.516376)
 		(stroke
 			(width 0.05)
@@
 		(layer "Edge.Cuts")
 	)
-	(gr_circle
-		(center 299.312324 178.65625)
-		(end 300.362324 178.65625)
-		(stroke
-			(width 0.05)
-			(type default)
-		)
-		(fill none)
-		(layer "Edge.Cuts")
-	)
 	(gr_line
 		(start 91.571875 69.5)
@@
 		(layer "Edge.Cuts")
 	)
+	(gr_circle
+		(center 146.912452 107.516376)
+		(end 147.962452 107.516376)
+		(stroke
+			(width 0.05)
+			(type default)
+		)
+		(fill none)
+		(layer "Edge.Cuts")
+	)
 	(gr_arc
 		(start 316.553132 69.5)
@@
 	)
 	(gr_circle
-		(center 108.812484 178.65625)
-		(end 109.862484 178.65625)
+		(center 261.212356 145.616344)
+		(end 262.262356 145.616344)
+		(stroke
+			(width 0.05)
+			(type default)
+		)
+		(fill none)
+		(layer "Edge.Cuts")
+	)
+	(gr_circle
+		(center 146.912452 145.616344)
+		(end 147.962452 145.616344)
 		(stroke
 			(width 0.05)
@@
 	)
 	(segment
+		(start 145.8875 109.6)
+		(end 145.8875 142.9375)
+		(width 0.2)
+		(layer "B.Cu")
+		(net 71)
+	)
+	(segment
 		(start 220.29458 84.001552)
 		(end 154.353852 84.001552)
@@
 	)
 	(segment
+		(start 145.8875 104.8375)
+		(end 144.53125 106.19375)
+		(width 0.2)
+		(layer "B.Cu")
+		(net 71)
+	)
+	(segment
 		(start 145.8875 92.467904)
 		(end 145.8875 96.275)
@@
 	)
 	(segment
-		(start 145.8875 172.475)
-		(end 145.8875 96.275)
+		(start 145.8875 147.7)
+		(end 145.8875 172.475)
+		(width 0.2)
+		(layer "B.Cu")
+		(net 71)
+	)
+	(segment
+		(start 144.53125 106.19375)
+		(end 144.53125 108.24375)
+		(width 0.2)
+		(layer "B.Cu")
+		(net 71)
+	)
+	(segment
+		(start 145.8875 142.9375)
+		(end 144.53125 144.29375)
+		(width 0.2)
+		(layer "B.Cu")
+		(net 71)
+	)
+	(segment
+		(start 144.53125 108.24375)
+		(end 145.8875 109.6)
+		(width 0.2)
+		(layer "B.Cu")
+		(net 71)
+	)
+	(segment
+		(start 144.53125 144.29375)
+		(end 144.53125 146.34375)
+		(width 0.2)
+		(layer "B.Cu")
+		(net 71)
+	)
+	(segment
+		(start 144.53125 146.34375)
+		(end 145.8875 147.7)
+		(width 0.2)
+		(layer "B.Cu")
+		(net 71)
+	)
+	(segment
+		(start 145.8875 96.275)
+		(end 145.8875 104.8375)
 		(width 0.2)
 		(layer "B.Cu")
@@
 	)
 	(segment
+		(start 258.83125 106.19375)
+		(end 258.83125 108.24375)
+		(width 0.2)
+		(layer "B.Cu")
+		(net 77)
+	)
+	(segment
+		(start 260.1875 104.8375)
+		(end 258.83125 106.19375)
+		(width 0.2)
+		(layer "B.Cu")
+		(net 77)
+	)
+	(segment
 		(start 239.225515 87.692487)
 		(end 242.380668 90.84764)
@@
 	)
 	(segment
+		(start 258.83125 146.34375)
+		(end 260.1875 147.7)
+		(width 0.2)
+		(layer "B.Cu")
+		(net 77)
+	)
+	(segment
 		(start 258.69922 90.84764)
 		(end 260.1875 92.33592)
@@
 	)
 	(segment
+		(start 260.1875 109.6)
+		(end 260.1875 142.9375)
+		(width 0.2)
+		(layer "B.Cu")
+		(net 77)
+	)
+	(segment
 		(start 242.380668 90.84764)
 		(end 258.69922 90.84764)
@@
 	)
 	(segment
-		(start 260.1875 172.475)
-		(end 260.1875 96.275)
-		(width 0.2)
-		(layer "B.Cu")
+		(start 260.1875 147.7)
+		(end 260.1875 172.475)
+		(width 0.2)
+		(layer "B.Cu")
+		(net 77)
+	)
+	(segment
+		(start 260.1875 142.9375)
+		(end 258.83125 144.29375)
+		(width 0.2)
+		(layer "B.Cu")
+		(net 77)
+	)
+	(segment
+		(start 258.83125 108.24375)
+		(end 260.1875 109.6)
+		(width 0.2)
+		(layer "B.Cu")
+		(net 77)
+	)
+	(segment
+		(start 258.83125 144.29375)
+		(end 258.83125 146.34375)
+		(width 0.2)
+		(layer "B.Cu")
+		(net 77)
+	)
+	(segment
+		(start 260.1875 96.275)
+		(end 260.1875 104.8375)
+		(width 0.2)
+		(layer "B.Cu")
