File: kicad/keyboard.kicad_sch (KiCad schematic)
At the start: 169 parts, among them SW1 Push, SW10 Push, SW11 Push, SW12 Push, SW13 Push, SW14 Push, SW15 Push, SW16 Push, SW17 Push, SW18 Push, SW19 Push, SW2 Push, SW20 Push, SW21 Push, SW22 Push, SW23 Push, SW24 Push, SW25 Push, SW26 Push, SW27 Push, SW28 Push, SW29 Push, SW3 Push, SW30 Push, SW31 Push, SW32 Push, SW33 Push, SW34 Push, SW35 Push, SW36 Push, SW37 Push, SW38 Push, SW39 Push, SW4 Push, SW40 Push, SW41 Push, SW42 Push, SW43 Push, SW44 Push, SW45 Push, SW46 Push, SW47 Push, SW48 Push, SW49 Push, SW5 Push, SW50 Push, SW51 Push, SW52 Push, SW53 Push, SW54 Push, SW55 Push, SW56 Push, SW57 Push, SW58 Push, SW59 Push, SW6 Push, SW60 Push, SW61 Push, SW62 Push, SW63 Push, SW64 Push, SW65 Push, SW66 Push, SW67 Push, SW68 Push, SW69 Push, SW7 Push, SW70 Push, SW71 Push, SW72 Push, SW73 Push, SW74 Push, SW75 Push, SW76 Push, SW77 Push, SW78 Push, SW79 Push, SW8 Push, SW80 Push, SW81 Push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

Commit message: 2
Parts:
- D1, D10, D11, D12, D13, D14, D15, D16, D17, D18, D19, D2, D20, D21, D22, D23, D24, D25, D26, D27, D28, D29, D3, D30, D31, D32, D33, D34, D35, D36, D37, D38, D39, D4, D40, D41, D42, D43, D44, D45, D46, D47, D48, D49, D5, D50, D51, D52, D53, D54, D55, D56, D57, D58, D59, D6, D60, D61, D62, D63, D64, D65, D66, D67, D68, D69, D7, D70, D71, D72, D73, D74, D75, D76, D77, D78, D79, D8, D80, D81, D82, D83, D84, D9: footprint MyLibrary:D1206 -> ScottoKeebs_Components:Diode_SOD-123
- SW1, SW10, SW11, SW12, SW13, SW14, SW15, SW16, SW17, SW18, SW19, SW2, SW20, SW21, SW22, SW23, SW24, SW25, SW26, SW27, SW28, SW29, SW3, SW30, SW31, SW32, SW33, SW34, SW35, SW36, SW37, SW38, SW39, SW4, SW40, SW41, SW42, SW43, SW44, SW45, SW46, SW47, SW48, SW49, SW5, SW50, SW51, SW52, SW53, SW54, SW55, SW56, SW57, SW58, SW59, SW6, SW60, SW61, SW62, SW63, SW64, SW65, SW66, SW67, SW68, SW69, SW7, SW70, SW71, SW72, SW73, SW74, SW75, SW76, SW77, SW78, SW79, SW8, SW80, SW81, SW82, SW83, SW84, SW9: footprint Library:Kailh_socket_PG1350 -> Gateron_KS33_Solderable:Gateron-KS33-Solderable-1U

Commit message: pi traces
Connections:
- net COL2: no longer U1.3 (GND)
- net ROW0: now also U1.27 (GPIO21); no longer U1.19 (GPIO14)
- net ROW1: now also U1.26 (GPIO20); no longer U1.20 (GPIO15)
- net ROW2: now also U1.25 (GPIO19); no longer U1.21 (GPIO16)
- net ROW3: now also U1.24 (GPIO18); no longer U1.22 (GPIO17)
- net ROW4: now also U1.22 (GPIO17); no longer U1.24 (GPIO18)
- net ROW5: now also U1.21 (GPIO16); no longer U1.25 (GPIO19)

Commit message: init
Parts:
- removed D13, D19, D25, D31, D37, D43, D49, D55, D61, D67, D7, D73, D74, D75, D76, D77, D78, D80, D81, D82, D83, D84: 1N47xxA, ScottoKeebs_Components:Diode_SOD-123, symbol Diode:1N47xxA
- removed SW13, SW19, SW25, SW31, SW37, SW43, SW49, SW55, SW61, SW67, SW7, SW73, SW74, SW75, SW76, SW77, SW78, SW80, SW81, SW82, SW83, SW84: Push, Gateron_KS33_Solderable:Gateron-KS33-Solderable-1U, symbol Switch:SW_Push
- removed U1: Raspberry_Pi_Pico, ScottoKeebs_MCU:Raspberry_Pi_Pico, symbol ScottoKeebs:MCU_Raspberry_Pi_Pico
- added U1: Arduino_Pro_Micro, ScottoKeebs_MCU:Arduino_Pro_Micro, symbol ScottoKeebs:MCU_Arduino_Pro_Micro
- SW1, SW10, SW11, SW12, SW14, SW15, SW16, SW17, SW18, SW2, SW20, SW21, SW22, SW23, SW24, SW26, SW27, SW28, SW29, SW3, SW30, SW32, SW33, SW34, SW35, SW36, SW38, SW39, SW4, SW40, SW41, SW42, SW44, SW45, SW46, SW47, SW48, SW5, SW50, SW51, SW52, SW53, SW54, SW56, SW57, SW58, SW59, SW6, SW60, SW62, SW63, SW64, SW65, SW66, SW68, SW69, SW70, SW71, SW72, SW79, SW8, SW9: footprint Gateron_KS33_Solderable:Gateron-KS33-Solderable-1U -> ScottoKeebs_Hotswap:Hotswap_Choc_V1_1.00u
Connections:
- net COL13 is gone; now on net COL11: SW79.2
- net COL0: now also U1.8 (5/PC6)
- net COL1: now also U1.7 (4/PD4)
- net COL10: now also U1.14 (16/PB2)
- net COL11: now also D79.2 (A), SW79.1, U1.13 (10/PB6)
- net COL2: now also U1.6 (3/PD0)
- net COL3: now also U1.5 (2/PD1)
- net COL4: now also U1.2 (RX1/PD2)
- net COL5: now also U1.1 (TX0/PD3)
- net COL6: now also U1.9 (6/PD7)
- net COL7: now also U1.10 (7/PE6)
- net COL8: now also U1.12 (9/PB5)
- net COL9: now also U1.11 (8/PB4)
- net ROW0: now also U1.17 (A0/PF7)
- net ROW1: now also U1.16 (15/PB1)
- net ROW2: now also U1.15 (14/PB3)
- net ROW3: now also U1.18 (A1/PF6)
- net ROW4: now also U1.19 (A2/PF5)
- net ROW5: now also U1.20 (A3/PF4)
Other:
- moved on the sheet: D79, SW79

Commit message: S67 fix
Parts:
- renumbered D79 to D67, SW79 to SW67
Connections:
- net COL11: no longer D67.2 (A), SW67.1
- new net: D67.2 (A), SW67.1
Changed lines of the file:
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@@
 	)
 	(junction
-		(at 233.68 49.53)
-		(diameter 0)
-		(color 0 0 0 0)
-	)
-	(junction
 		(at 243.84 49.53)
 		(diameter 0)
@@
 	(wire
 		(pts
-			(xy 233.68 49.53) (xy 243.84 49.53)
-		)
-		(stroke
-			(width 0)
-			(type default)
-		)
-	)
-	(wire
-		(pts
 			(xy 129.54 72.39) (xy 129.54 83.82)
 		)
@@
 		(on_board yes)
 		(dnp no)
-		(property "Reference" "SW79"
+		(property "Reference" "SW67"
 			(at 238.76 52.07 0)
 			(effects
@@
 			(project "keyboard"
 				(path "/4342f055-467b-4789-a8ed-b19f1b214d4d"
-					(reference "SW79")
+					(reference "SW67")
 					(unit 1)
 				)
@@
 		(on_board yes)
 		(dnp no)
-		(property "Reference" "D79"
+		(property "Reference" "D67"
 			(at 236.22 55.88 90)
 			(effects
@@
 			(project "keyboard"
 				(path "/4342f055-467b-4789-a8ed-b19f1b214d4d"
-					(reference "D79")
+					(reference "D67")
 					(unit 1)
 				)

Commit message: spacebar
Parts:
- removed D36: 1N47xxA, ScottoKeebs_Components:Diode_SOD-123, symbol Diode:1N47xxA
- removed SW36: Push, ScottoKeebs_Hotswap:Hotswap_Choc_V1_1.00u, symbol Switch:SW_Push
Other:
- moved on the sheet: D42, SW42
Changed lines of the file:
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@@
 	)
 	(junction
-		(at 157.48 114.3)
-		(diameter 0)
-		(color 0 0 0 0)
-	)
-	(junction
 		(at 119.38 68.58)
 		(diameter 0)
@@
 	)
 	(junction
-		(at 167.64 95.25)
-		(diameter 0)
-		(color 0 0 0 0)
-	)
-	(junction
 		(at 167.64 60.96)
 		(diameter 0)
@@
 	)
 	(junction
-		(at 170.18 114.3)
+		(at 163.83 114.3)
 		(diameter 0)
 		(color 0 0 0 0)
@@
 	)
 	(junction
-		(at 167.64 106.68)
-		(diameter 0)
-		(color 0 0 0 0)
-	)
-	(junction
 		(at 129.54 72.39)
 		(diameter 0)
@@
 	(wire
 		(pts
-			(xy 129.54 45.974) (xy 129.54 60.96)
+			(xy 180.34 106.68) (xy 180.34 95.25)
 		)
 		(stroke
@@
 	(wire
 		(pts
-			(xy 205.74 45.974) (xy 205.74 60.96)
+			(xy 129.54 45.974) (xy 129.54 60.96)
 		)
 		(stroke
@@
 	(wire
 		(pts
-			(xy 208.28 91.44) (xy 220.98 91.44)
+			(xy 205.74 45.974) (xy 205.74 60.96)
 		)
 		(stroke
@@
 	(wire
 		(pts
-			(xy 231.14 72.39) (xy 231.14 83.82)
+			(xy 208.28 91.44) (xy 220.98 91.44)
 		)
 		(stroke
@@
 	(wire
 		(pts
-			(xy 104.14 72.39) (xy 104.14 83.82)
+			(xy 231.14 72.39) (xy 231.14 83.82)
 		)
 		(stroke
@@
 	(wire
 		(pts
-			(xy 180.34 95.25) (xy 180.34 106.68)
+			(xy 104.14 72.39) (xy 104.14 83.82)
 		)
 		(stroke
@@
 	(wire
 		(pts
-			(xy 157.48 114.3) (xy 170.18 114.3)
-		)
-		(stroke
-			(width 0)
-			(type default)
-		)
-	)
-	(wire
-		(pts
 			(xy 170.18 68.58) (xy 182.88 68.58)
 		)
@@
 	(wire
 		(pts
-			(xy 167.64 106.68) (xy 167.64 106.934)
+			(xy 173.99 106.68) (xy 180.34 106.68)
 		)
 		(stroke
@@
 	(wire
 		(pts
-			(xy 144.78 114.3) (xy 157.48 114.3)
+			(xy 144.78 114.3) (xy 163.83 114.3)
 		)
 		(stroke
@@
 	(wire
 		(pts
-			(xy 170.18 114.3) (xy 182.88 114.3)
+			(xy 163.83 114.3) (xy 182.88 114.3)
 		)
 		(stroke
@@
 	(wire
 		(pts
-			(xy 167.64 95.25) (xy 167.64 106.68)
-		)
-		(stroke
-			(width 0)
-			(type default)
-		)
-	)
-	(wire
-		(pts
 			(xy 92.71 80.01) (xy 93.98 80.01)
 		)
@@
 	)
 	(symbol
-		(lib_id "Switch:SW_Push")
-		(at 162.56 106.68 0)
-		(unit 1)
-		(exclude_from_sim no)
-		(in_bom yes)
-		(on_board yes)
-		(dnp no)
-		(property "Reference" "SW36"
-			(at 162.56 109.22 0)
-			(effects
-				(font
-					(size 1.27 1.27)
-				)
-			)
-		)
-		(property "Value" "Push"
-			(at 162.56 101.7524 0)
-			(effects
-				(font
-					(size 1.27 1.27)
-				)
-				(hide yes)
-			)
-		)
-		(property "Footprint" "ScottoKeebs_Hotswap:Hotswap_Choc_V1_1.00u"
-			(at 162.56 101.6 0)
-			(effects
-				(font
-					(size 1.27 1.27)
-				)
-				(hide yes)
-			)
-		)
-		(property "Datasheet" "~"
-			(at 162.56 101.6 0)
-			(effects
-				(font
-					(size 1.27 1.27)
-				)
-				(hide yes)
-			)
-		)
-		(property "Description" ""
-			(at 162.56 106.68 0)
-			(effects
-				(font
-					(size 1.27 1.27)
-				)
-				(hide yes)
-			)
-		)
-		(pin "1"
-		)
-		(pin "2"
-		)
-		(instances
-			(project "keyboard"
-				(path "/4342f055-467b-4789-a8ed-b19f1b214d4d"
-					(reference "SW36")
-					(unit 1)
-				)
-			)
-		)
-	)
-	(symbol
 		(lib_id "Diode:1N47xxA")
 		(at 132.08 87.63 90)
@@
 	(symbol
 		(lib_id "Diode:1N47xxA")
-		(at 170.18 110.49 90)
+		(at 163.83 110.49 90)
 		(unit 1)
 		(exclude_from_sim no)
@@
 		(dnp no)
 		(property "Reference" "D42"
-			(at 172.72 113.03 90)
+			(at 166.37 113.03 90)
 			(effects
 				(font
@@
 		)
 		(property "Value" "1N47xxA"
-			(at 172.72 111.7599 90)
+			(at 166.37 111.7599 90)
 			(effects
 				(font
@@
 		)
 		(property "Footprint" "ScottoKeebs_Components:Diode_SOD-123"
-			(at 174.625 110.49 0)
+			(at 168.275 110.49 0)
 			(effects
 				(font
@@
 		)
 		(property "Datasheet" "https://www.vishay.com/docs/85816/1n4728a.pdf"
-			(at 170.18 110.49 0)
+			(at 163.83 110.49 0)
 			(effects
 				(font
@@
 		)
 		(property "Description" ""
-			(at 170.18 110.49 0)
+			(at 163.83 110.49 0)
 			(effects
 				(font
@@
 	(symbol
 		(lib_id "Switch:SW_Push")
-		(at 175.26 106.68 0)
+		(at 168.91 106.68 0)
 		(unit 1)
 		(exclude_from_sim no)
@@
 		(dnp no)
 		(property "Reference" "SW42"
-			(at 175.26 109.22 0)
+			(at 168.91 109.22 0)
 			(effects
 				(font
@@
 		)
 		(property "Value" "Push"
-			(at 175.26 101.7524 0)
+			(at 168.91 101.7524 0)
 			(effects
 				(font
@@
 		)
 		(property "Footprint" "ScottoKeebs_Hotswap:Hotswap_Choc_V1_1.00u"
-			(at 175.26 101.6 0)
+			(at 168.91 101.6 0)
 			(effects
 				(font
@@
 		)
 		(property "Datasheet" "~"
-			(at 175.26 101.6 0)
+			(at 168.91 101.6 0)
 			(effects
 				(font
@@
 		)
 		(property "Description" ""
-			(at 175.26 106.68 0)
+			(at 168.91 106.68 0)
 			(effects
 				(font
@@
 					(unit 1)
 				)
-			)
-		)
-	)
-	(symbol
-		(lib_id "Diode:1N47xxA")
-		(at 157.48 110.49 90)
-		(unit 1)
-		(exclude_from_sim no)
-		(in_bom yes)
-		(on_board yes)
-		(dnp no)
-		(property "Reference" "D36"
-			(at 160.02 113.03 90)
-			(effects
-				(font
-					(size 1.27 1.27)
-				)
-				(justify right)
-			)
-		)
-		(property "Value" "1N47xxA"
-			(at 160.02 111.7599 90)
-			(effects
-				(font
-					(size 1.27 1.27)
-				)
-				(justify right)
-				(hide yes)
-			)
-		)
-		(property "Footprint" "ScottoKeebs_Components:Diode_SOD-123"
-			(at 161.925 110.49 0)
-			(effects
-				(font
-					(size 1.27 1.27)
-				)
-				(hide yes)
-			)
-		)
-		(property "Datasheet" "https://www.vishay.com/docs/85816/1n4728a.pdf"
-			(at 157.48 110.49 0)
-			(effects
-				(font
-					(size 1.27 1.27)
-				)
-				(hide yes)
-			)
-		)
-		(property "Description" ""
-			(at 157.48 110.49 0)
-			(effects
-				(font
-					(size 1.27 1.27)
-				)
-				(hide yes)
-			)
-		)
-		(pin "1"
-		)
-		(pin "2"
-		)
-		(instances
-			(project "keyboard"
-				(path "/4342f055-467b-4789-a8ed-b19f1b214d4d"
-					(reference "D36")
-					(unit 1)
-				)
