File: pcb/keyboard.kicad_pcb (KiCad board)
At the start: 2 copper layers, 232.6 x 118.3 mm, 123 parts, among them SW1 Push, SW10 Push, SW11 Push, SW12 Push, SW14 Push, SW15 Push, SW16 Push, SW17 Push, SW18 Push, SW2 Push, SW20 Push, SW21 Push, SW22 Push, SW23 Push, SW24 Push, SW26 Push, SW27 Push, SW28 Push, SW29 Push, SW3 Push, SW30 Push, SW32 Push, SW33 Push, SW34 Push, SW35 Push, SW38 Push, SW39 Push, SW4 Push, SW40 Push, SW41 Push, SW42 Push, SW44 Push, SW45 Push, SW46 Push, SW47 Push, SW48 Push, SW5 Push, SW50 Push, SW51 Push, SW52 Push, SW53 Push, SW54 Push, SW56 Push, SW57 Push, SW58 Push, SW59 Push, SW6 Push, SW60 Push, SW62 Push, SW63 Push, SW64 Push, SW65 Push, SW66 Push, SW67 Push, SW68 Push, SW69 Push, SW70 Push, SW71 Push, SW72 Push, SW8 Push, SW9 Push, U1 Arduino_Pro_Micro

Commit message: production edits
Routing:
- added copper zone on B.Cu, net (none)
- added copper zone on F.Cu, net (none)
Changed lines of the file:
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@@
 		(net 83)
+	)
+	(zone
+		(net 0)
+		(net_name "")
+		(layers "F&B.Cu")
+		(hatch edge 0.5)
+		(connect_pads
+			(clearance 0.5)
+		)
+		(min_thickness 0.25)
+		(filled_areas_thickness no)
+		(fill yes
+			(thermal_gap 0.5)
+			(thermal_bridge_width 0.5)
+			(island_removal_mode 1)
+			(island_area_min 10)
+		)
+		(polygon
+			(pts
+				(xy 71.903125 56.021875) (xy 330.26875 56.021875) (xy 330.26875 196.515625) (xy 75.475 196.515625)
+			)
+		)
 	)
 	(group ""
