File: source/kicad_choc_v1/krtkus.kicad_pcb (KiCad board)
At the start: 2 copper layers, 232.6 x 118.3 mm, 123 parts, among them SW1 Push, SW10 Push, SW11 Push, SW12 Push, SW14 Push, SW15 Push, SW16 Push, SW17 Push, SW18 Push, SW2 Push, SW20 Push, SW21 Push, SW22 Push, SW23 Push, SW24 Push, SW26 Push, SW27 Push, SW28 Push, SW29 Push, SW3 Push, SW30 Push, SW32 Push, SW33 Push, SW34 Push, SW35 Push, SW38 Push, SW39 Push, SW4 Push, SW40 Push, SW41 Push, SW42 Push, SW44 Push, SW45 Push, SW46 Push, SW47 Push, SW48 Push, SW5 Push, SW50 Push, SW51 Push, SW52 Push, SW53 Push, SW54 Push, SW56 Push, SW57 Push, SW58 Push, SW59 Push, SW6 Push, SW60 Push, SW62 Push, SW63 Push, SW64 Push, SW65 Push, SW66 Push, SW67 Push, SW68 Push, SW69 Push, SW70 Push, SW71 Push, SW72 Push, SW8 Push, SW9 Push, U1 Arduino_Pro_Micro

Commit message: unification
Parts:
- moved U1 9.16 mm to (234.4, 80.6)
Routing:
- net COL11: track 208.9 -> 198.6 mm
- net COL10: track 175.1 -> 165.0 mm
- net ROW1: track 370.5 -> 361.2 mm
- net ROW2: track 389.8 -> 380.5 mm
- net COL4: track 133.0 -> 142.4 mm
- net COL3: track 160.6 -> 169.9 mm
- net COL2: track 181.7 -> 191.1 mm
- net COL1: track 204.6 -> 214.0 mm
- net COL0: track 242.9 -> 252.3 mm
- net COL8: track 121.6 -> 112.2 mm
- net ROW4: track 470.2 -> 479.2 mm
- net ROW5: track 484.6 -> 493.6 mm
- net ROW3: track 451.3 -> 460.4 mm
- net COL9: track 148.0 -> 139.0 mm
- net COL5: track 86.8 -> 95.8 mm
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